Commit message: chore: adapt moveit_config package to use the new franka_description package

File: franka_fr3_moveit_config/srdf/fr3_arm.xacro (robot description, xacro)
@@ -1,6 +1,6 @@
 <?xml version="1.0" ?>
-<robot xmlns:xacro="http://www.ros.org/wiki/xacro" name="panda">
-  <xacro:macro name="panda_arm" params="arm_id:='panda' ">
-    <xacro:include filename="$(find franka_moveit_config)/srdf/group_definition.xacro"/>
+<robot xmlns:xacro="http://www.ros.org/wiki/xacro" name="fr3">
+  <xacro:macro name="fr3_arm" params="arm_id:='fr3' ">
+    <xacro:include filename="$(find franka_fr3_moveit_config)/srdf/group_definition.xacro"/>
     <xacro:group_definition arm_id="${arm_id}" group_name="${arm_id}_manipulator" tip_link="${arm_id}_hand_tcp"/>
     <xacro:group_definition arm_id="${arm_id}" group_name="${arm_id}_arm" tip_link="${arm_id}_link8"/>

File: franka_fr3_moveit_config/srdf/fr3_arm_hand.xacro (robot description, xacro)
@@ -1,5 +1,5 @@
 <?xml version='1.0' encoding='utf-8'?>
-<robot xmlns:xacro="http://www.ros.org/wiki/xacro" name="panda">
-  <xacro:macro name="panda_arm_hand" params="arm_id:='panda' ">
+<robot xmlns:xacro="http://www.ros.org/wiki/xacro" name="fr3">
+  <xacro:macro name="fr3_arm_hand" params="arm_id:='fr3' ">
     <group_state name="open" group="hand">
       <joint name="${arm_id}_finger_joint1" value="0.035"/>

File: franka_fr3_moveit_config/srdf/group_definition.xacro (robot description, xacro)
@@ -1,4 +1,4 @@
 <?xml version="1.0" encoding="UTF-8"?>
-<robot xmlns:xacro="http://www.ros.org/wiki/xacro" name="panda">
+<robot xmlns:xacro="http://www.ros.org/wiki/xacro" name="fr3">
   <xacro:macro name="group_definition" params="group_name arm_id tip_link">
     <group name="${group_name}">

File: franka_fr3_moveit_config/srdf/hand.xacro (robot description, xacro)
@@ -1,5 +1,5 @@
 <?xml version="1.0" ?>
-<robot xmlns:xacro="http://www.ros.org/wiki/xacro" name="panda">
-  <xacro:macro name="hand" params="arm_id:='panda' ">
+<robot xmlns:xacro="http://www.ros.org/wiki/xacro" name="fr3">
+  <xacro:macro name="hand" params="arm_id:='fr3' ">
     <group name="hand">
       <link name="${arm_id}_hand"/>
